Commit message: Update ros2_ws MoveIt/Fabric config and add mujoco bridge

File: MarvinDocker/ros2_ws/src/Marvin-description/urdf/marvin_CCS_m6.urdf.xacro (robot description, xacro)
@@ -7,7 +7,7 @@
   <xacro:arg name="gripper_debug" default="false" />
   <xacro:property name="left_gripper_mount_xyz" value="0 0 0" />
-  <xacro:property name="left_gripper_mount_rpy" value="0 0 0" />
+  <xacro:property name="left_gripper_mount_rpy" value="0 0 -1.5708" />
   <xacro:property name="right_gripper_mount_xyz" value="0 0 0" />
-  <xacro:property name="right_gripper_mount_rpy" value="0 0 0" />
+  <xacro:property name="right_gripper_mount_rpy" value="0 0 -1.5708" />
   <xacro:property name="left_tool_base_x" value="${-0.0116961}" />
   <xacro:property name="left_tool_base_y" value="${-0.0901059}" />
